Commit message: Done: Rotation planche cmd vitesse

File: robot_description/src/description/robot_description.urdf (robot description, URDF)
Before this commit: robot sam_bot, 14 links, 13 joints
Links:
- added link my_pivot; collision box size=0.7 0.05 0.2; visual box size=0.7 0.05 0.2
Joints:
- added joint my_pivot_joint: type revolute, parent base_link, child my_pivot, origin xyz=1 0.0 0 rpy=0 0 0, axis 1 0 0, limit lower=0 upper=0.38 effort=1000.0 velocity=10

Commit message: Pb

File: robot_description/src/description/robot_description.urdf (robot description, URDF)
Before this commit: robot sam_bot, 15 links, 14 joints
Links:
- removed link my_pivot
- link segment_central: geometry visual box size=0.7 0.05 0.2
- link segment_d1: geometry visual box size=0.3 0.05 0.2
- link segment_d2: geometry visual box size=0.3 0.05 0.2
- link segment_d3: geometry visual box size=0.3 0.05 0.2
- link segment_g1: geometry visual box size=0.3 0.05 0.2
- link segment_g2: geometry visual box size=0.3 0.05 0.2
- link segment_g3: geometry visual box size=0.3 0.05 0.2
- link segment_triangled: geometry visual box size=0.3 0.05 0.2
- link segment_triangleg: geometry visual box size=0.3 0.05 0.2
Joints:
- removed joint my_pivot_joint
- joint segment_central_joint: axis (none) -> 1 0 0; limit (none) -> lower=0 upper=10000000 effort=10000000.0 velocity=30; origin xyz=0.25 0.0 0 rpy=0 0 ${0.5 * pi} -> xyz=0.25 0.0 0 rpy=-1.5 0 ${-0.5 * pi}; type fixed -> revolute
