Commit message: Done : Motorisation et non commande

File: robot_description/src/description/collector/collector.xacro (robot description, xacro)
@@ -3,6 +3,63 @@
     xmlns:xacro="http://ros.org/wiki/xacro">
     <xacro:include filename="$(find robot_description)/src/description/collector/segment.xacro" />
+    <gazebo>
+        <plugin filename="libgazebo_ros2_control.so" name="gazebo_ros2_control">
+        <parameters>$(find gazebo_ros2_control_demos)/config/gripper_controller.yaml</parameters>
+        </plugin>
+    </gazebo>
     <xacro:macro name="collector">
-        <xacro:segment name="segment_central" x="0.7" y="0.05" z="0.2" joint_parent="base_link" joint_origin_xyz="0.25 0.0 0" joint_origin_rpy="0 0 ${0.5 * pi}"/>
+        <!-- <xacro:segment name="segment_central" x="0.7" y="0.05" z="0.2" joint_parent="base_link" joint_origin_xyz="0.25 0.0 0" joint_origin_rpy="0 0 ${0.5 * pi}"/> -->
+        <gazebo reference="segment_central">
+            <visual>
+            <material>
+            <ambient>1. 0.3 0.3 1.0</ambient>
+            <diffuse>1. 0.3 0.3 1.0</diffuse>
+            <specular>1. 0.3 0.3 1.0</specular>
+            <emissive>1. 0.3 0.3 1.0</emissive>
+            </material>
+            </visual>
+        </gazebo>
+        <link name="segment_central">
+            <visual>
+            <geometry>
+                <box size="0.7 0.05 0.2"/>
+            </geometry>
+            <material name="Brown">
+                <color rgba="0.30 0.15 0.0 1.0"/>
+            </material>
+            </visual>
+            <!-- <collision>
+            <origin xyz="0 0 0" rpy="0 0 0"/>
+            <geometry>0 0.0 0.0 1.0
+                <box size="0.7 0.05 0.2"/>
+            </geometry>
+            </collision> -->
+            <xacro:box_inertia m="0.1" w="0.7" d="0.05" h="0.2"/>
+        </link>
+        <!-- <joint name="segment_central_joint" type="fixed">
+            <parent link="base_link"/>
+            <child link="segment_central"/>
+            <origin xyz="0.25 0.0 0" rpy="0 0 ${0.5 * pi}"/>
+        </joint> -->
+        <joint name="segment_central_joint" type="revolute">
+            <axis xyz="0 1 0"/>
+            <origin xyz="0.25 0.0 0" rpy="-1.5 0 ${-0.5 * pi}"/>
+            <parent link="base_link"/>
+            <child link="segment_central"/>
+            <limit effort="10000.0" lower="0" upper="0.1" velocity="0"/>
+        </joint>
+        <ros2_control name="GazeboSystem" type="system">
+                <hardware>
+                <plugin>gazebo_ros2_control/GazeboSystem</plugin>
+                </hardware>
+                <joint name="segment_central_joint">
+                <command_interface name="position"/>
+                <state_interface name="position">
+                    <param name="initial_value">0.0</param>
+                </state_interface>
+                <state_interface name="velocity"/>
+                <state_interface name="effort"/>
+                </joint>
+            </ros2_control>
         <xacro:segment name="segment_d1" x="0.3" y="0.05" z="0.2" joint_parent="segment_central" joint_origin_xyz="-.25 -.32 0" joint_origin_rpy="0 0 ${0.16 * pi}"/>
         <xacro:segment name="segment_d2" x="0.3" y="0.05" z="0.2" joint_parent="segment_d1" joint_origin_xyz="-0.30 -0.07 0" joint_origin_rpy="0 0 ${0.16 * pi}"/>

File: robot_description/src/description/collector/segment_central.xacro (robot description, xacro)
@@ -22,17 +22,42 @@
                 </material>
             </visual>
-            <!-- <collision>
+            <collision>
                 <origin xyz="0 0 0" rpy="0 0 0"/>
                 <geometry>0 0.0 0.0 1.0
                     <box size="${x} ${y} ${z}"/>
                 </geometry>
-            </collision> -->
+            </collision>
             <xacro:box_inertia m="0.1" w="${x}" d="${y}" h="${z}"/>
         </link>
-        <joint name="${name}_joint" type="fixed">
+        <!-- <joint name="${name}_joint" type="fixed">
             <parent link="${joint_parent}"/>
             <child link="${name}"/>
             <origin xyz="${joint_origin_xyz}" rpy="${joint_origin_rpy}"/>
-        </joint>
+        </joint> -->
+        <!-- <joint name="segment_central_joint" type="revolute">
+            <axis xyz="1 0 0"/>
+            <origin xyz="0.25 0.0 0" rpy="-1.5 0 ${-0.5 * pi}"/>
+            <parent link="base_link"/>
+            <child link="segment_central"/>
+            <limit effort="10000000.0" lower="0" upper="10000000" velocity="30"/>
+        </joint>  -->
+        <!-- <ros2_control name="GazeboSystem" type="system">
+            <hardware>
+            <plugin>gazebo_ros2_control/GazeboSystem</plugin>
+            </hardware>
+            <joint name="segment_central_joint">
+            <command_interface name="velocity"/>
+            <state_interface name="velocity">
+                <param name="initial_value">0.0</param>
+            </state_interface>
+            <state_interface name="velocity"/>
+            <state_interface name="effort"/>
+            </joint>
+        </ros2_control>
+        <gazebo>
+            <plugin filename="libgazebo_ros2_control.so" name="gazebo_ros2_control">
+            <parameters>$(find gazebo_ros2_control_demos)/config/gripper_controller.yaml</parameters>
+            </plugin>
+        </gazebo> -->
     </xacro:macro>
 </robot>

Commit message: Done: Control pince, pb collision et inertie

File: robot_description/src/description/collector/collector.xacro (robot description, xacro)
@@ -3,9 +3,9 @@
     xmlns:xacro="http://ros.org/wiki/xacro">
     <xacro:include filename="$(find robot_description)/src/description/collector/segment.xacro" />
-    <gazebo>
+    <!-- <gazebo>
         <plugin filename="libgazebo_ros2_control.so" name="gazebo_ros2_control">
         <parameters>$(find gazebo_ros2_control_demos)/config/gripper_controller.yaml</parameters>
         </plugin>
-    </gazebo>
+    </gazebo> -->
     <xacro:macro name="collector">
         <!-- <xacro:segment name="segment_central" x="0.7" y="0.05" z="0.2" joint_parent="base_link" joint_origin_xyz="0.25 0.0 0" joint_origin_rpy="0 0 ${0.5 * pi}"/> -->
@@ -42,5 +42,5 @@
             <origin xyz="0.25 0.0 0" rpy="0 0 ${0.5 * pi}"/>
         </joint> -->
-        <joint name="segment_central_joint" type="revolute">
+        <!-- <joint name="segment_central_joint" type="revolute">
             <axis xyz="0 1 0"/>
             <origin xyz="0.25 0.0 0" rpy="-1.5 0 ${-0.5 * pi}"/>
@@ -48,18 +48,41 @@
             <child link="segment_central"/>
             <limit effort="10000.0" lower="0" upper="0.1" velocity="0"/>
+        </joint>  -->
+        <joint name="segment_central_joint" type="revolute">
+            <axis xyz="1 0 0"/>
+            <origin xyz="0.25 0.0 0" rpy="-1.5 0 ${-0.5 * pi}"/>
+            <parent link="base_link"/>
+            <child link="segment_central"/>
+            <limit effort="1000.0" lower="-0.15" upper="0.15" velocity="30"/>
+            <!-- <dynamics damping="0.0" friction="0.0"/> -->
         </joint>
         <ros2_control name="GazeboSystem" type="system">
-                <hardware>
-                <plugin>gazebo_ros2_control/GazeboSystem</plugin>
-                </hardware>
-                <joint name="segment_central_joint">
-                <command_interface name="position"/>
-                <state_interface name="position">
-                    <param name="initial_value">0.0</param>
-                </state_interface>
+            <hardware>
+            <plugin>gazebo_ros2_control/GazeboSystem</plugin>
+            </hardware>
+            <!-- <joint name="segment_central_joint">
+            <command_interface name="position"/>
+            <state_interface name="position">
+                <param name="initial_value">0.0</param>
+            </state_interface>
+            <state_interface name="velocity"/>
+            <state_interface name="effort"/>
+            </joint> -->
+            <joint name="segment_central_joint">
+                <command_interface name="velocity">
+                    <param name="min">-0.10</param>
+                    <param name="max">0.10</param>
+                </command_interface>
+                <state_interface name="position"/>
                 <state_interface name="velocity"/>
                 <state_interface name="effort"/>
-                </joint>
-            </ros2_control>
+            </joint>
+        </ros2_control>
+        <gazebo>
+            <plugin filename="libgazebo_ros2_control.so" name="gazebo_ros2_control">
+            <parameters>/home/mirado/ws_CollecteBalle/src/CollecteBalle/config/gripper_controller.yaml</parameters>
+            <!-- <parameters>$(find CollecteBalle)/config/gripper_controller.yaml</parameters> -->
+            </plugin>
+        </gazebo>
         <xacro:segment name="segment_d1" x="0.3" y="0.05" z="0.2" joint_parent="segment_central" joint_origin_xyz="-.25 -.32 0" joint_origin_rpy="0 0 ${0.16 * pi}"/>
         <xacro:segment name="segment_d2" x="0.3" y="0.05" z="0.2" joint_parent="segment_d1" joint_origin_xyz="-0.30 -0.07 0" joint_origin_rpy="0 0 ${0.16 * pi}"/>

Commit message: Modif readme

File: robot_description/src/description/collector/collector.xacro (robot description, xacro)
@@ -3,9 +3,4 @@
     xmlns:xacro="http://ros.org/wiki/xacro">
     <xacro:include filename="$(find robot_description)/src/description/collector/segment.xacro" />
-    <!-- <gazebo>
-        <plugin filename="libgazebo_ros2_control.so" name="gazebo_ros2_control">
-        <parameters>$(find gazebo_ros2_control_demos)/config/gripper_controller.yaml</parameters>
-        </plugin>
-    </gazebo> -->
     <xacro:macro name="collector">
         <!-- <xacro:segment name="segment_central" x="0.7" y="0.05" z="0.2" joint_parent="base_link" joint_origin_xyz="0.25 0.0 0" joint_origin_rpy="0 0 ${0.5 * pi}"/> -->
@@ -37,16 +32,4 @@
             <xacro:box_inertia m="0.1" w="0.7" d="0.05" h="0.2"/>
         </link>
-        <!-- <joint name="segment_central_joint" type="fixed">
-            <parent link="base_link"/>
-            <child link="segment_central"/>
-            <origin xyz="0.25 0.0 0" rpy="0 0 ${0.5 * pi}"/>
-        </joint> -->
-        <!-- <joint name="segment_central_joint" type="revolute">
-            <axis xyz="0 1 0"/>
-            <origin xyz="0.25 0.0 0" rpy="-1.5 0 ${-0.5 * pi}"/>
-            <parent link="base_link"/>
-            <child link="segment_central"/>
-            <limit effort="10000.0" lower="0" upper="0.1" velocity="0"/>
-        </joint>  -->
         <joint name="segment_central_joint" type="revolute">
             <axis xyz="1 0 0"/>
@@ -61,12 +44,4 @@
             <plugin>gazebo_ros2_control/GazeboSystem</plugin>
             </hardware>
-            <!-- <joint name="segment_central_joint">
-            <command_interface name="position"/>
-            <state_interface name="position">
-                <param name="initial_value">0.0</param>
-            </state_interface>
-            <state_interface name="velocity"/>
-            <state_interface name="effort"/>
-            </joint> -->
             <joint name="segment_central_joint">
                 <command_interface name="velocity">
@@ -81,6 +56,5 @@
         <gazebo>
             <plugin filename="libgazebo_ros2_control.so" name="gazebo_ros2_control">
-            <parameters>/home/mirado/ws_CollecteBalle/src/CollecteBalle/config/gripper_controller.yaml</parameters>
-            <!-- <parameters>$(find CollecteBalle)/config/gripper_controller.yaml</parameters> -->
+            <parameters>$(find robot_description)/config/gripper_controller.yaml</parameters>
             </plugin>
         </gazebo>
