Commit message: mise en forme PeP8

File: robot_description/src/description/collector/segment_central.xacro (robot description, xacro)
@@ -16,17 +16,16 @@
             <visual>
                 <geometry>
-                    <box size="${x} ${y} ${z}"/>
+                    <box size="${x} ${y} ${z}" />
                 </geometry>
                 <material name="Brown">
-                    <color rgba="0.30 0.15 0.0 1.0"/>
+                    <color rgba="0.30 0.15 0.0 1.0" />
                 </material>
             </visual>
             <collision>
-                <origin xyz="0 0 0" rpy="0 0 0"/>
-                <geometry>0 0.0 0.0 1.0
-                    <box size="${x} ${y} ${z}"/>
+                <origin xyz="0 0 0" rpy="0 0 0" />
+                <geometry>0 0.0 0.0 1.0 <box size="${x} ${y} ${z}" />
                 </geometry>
             </collision>
-            <xacro:box_inertia m="0.1" w="${x}" d="${y}" h="${z}"/>
+            <xacro:box_inertia m="0.1" w="${x}" d="${y}" h="${z}" />
         </link>
         <!-- <joint name="${name}_joint" type="fixed">

File: robot_description/src/description/robot_description.xacro (robot description, xacro)
@@ -2,5 +2,6 @@
 <robot name="roballos"
   xmlns:xacro="http://ros.org/wiki/xacro">
-  <xacro:include filename="$(find robot_description)/src/description/robot_parts/collector/collector.xacro" />
+  <xacro:include
+    filename="$(find robot_description)/src/description/robot_parts/collector/collector.xacro" />
   <xacro:include filename="$(find robot_description)/src/description/robot_parts/property.xacro" />
   <xacro:include filename="$(find robot_description)/src/description/robot_parts/base.xacro" />
@@ -9,9 +10,9 @@
   <xacro:include filename="$(find robot_description)/src/description/robot_parts/caster_wheel.xacro" />
   <xacro:include filename="$(find robot_description)/src/description/robot_parts/control.xacro" />
-  <xacro:base/>
-  <xacro:battery/>
-  <xacro:wheels/>
-  <xacro:caster_wheel/>
-  <xacro:collector/>
-  <xacro:control/>
+  <xacro:base />
+  <xacro:battery />
+  <xacro:wheels />
+  <xacro:caster_wheel />
+  <xacro:collector />
+  <xacro:control />
 </robot>

File: robot_description/src/description/robot_parts/base.xacro (robot description, xacro)
@@ -18,25 +18,27 @@
                 <origin xyz="-0.2 -0.15 0" rpy="${pi/2} 0 0" />
                 <geometry>
-                    <mesh filename="$(find robot_description)/src/description/robot_parts/meshes/chassis_is.dae" scale="0.001 0.001 0.001"/>
+                    <mesh
+                        filename="$(find robot_description)/src/description/robot_parts/meshes/chassis_is.dae"
+                        scale="0.001 0.001 0.001" />
                 </geometry>
                 <material name="Cyan">
-                    <color rgba="0 1.0 1.0 1.0"/>
+                    <color rgba="0 1.0 1.0 1.0" />
                 </material>
             </visual>
             <collision>
                 <geometry>
-                    <box size="${base_length} ${base_width} ${base_height}"/>
+                    <box size="${base_length} ${base_width} ${base_height}" />
                 </geometry>
             </collision>
-            <xacro:box_inertia m="15" w="${base_width}" d="${base_length}" h="${base_height}"/>
+            <xacro:box_inertia m="15" w="${base_width}" d="${base_length}" h="${base_height}" />
         </link>
         <!-- Robot Footprint -->
         <link name="base_footprint">
-            <xacro:box_inertia m="0" w="0" d="0" h="0"/>
+            <xacro:box_inertia m="0" w="0" d="0" h="0" />
         </link>
         <joint name="base_joint" type="fixed">
-            <parent link="base_link"/>
-            <child link="base_footprint"/>
-            <origin xyz="0.0 0.0 ${-(wheel_radius+wheel_zoff)}" rpy="0 0 0"/>
+            <parent link="base_link" />
+            <child link="base_footprint" />
+            <origin xyz="0.0 0.0 ${-(wheel_radius+wheel_zoff)}" rpy="0 0 0" />
         </joint>
     </xacro:macro>

File: robot_description/src/description/robot_parts/battery.xacro (robot description, xacro)
@@ -17,21 +17,21 @@
             <visual>
                 <geometry>
-                    <box size="0.1 0.2 0.1"/>
+                    <box size="0.1 0.2 0.1" />
                 </geometry>
                 <material name="Cyan">
-                    <color rgba="0 1.0 1.0 1.0"/>
+                    <color rgba="0 1.0 1.0 1.0" />
                 </material>
             </visual>
             <collision>
                 <geometry>
-                    <box size="0.1 0.2 0.1"/>
+                    <box size="0.1 0.2 0.1" />
                 </geometry>
             </collision>
-            <xacro:box_inertia m="5" w="0.1" d="0.2" h="0.1"/>
+            <xacro:box_inertia m="5" w="0.1" d="0.2" h="0.1" />
         </link>
         <joint name="battery_joint" type="fixed">
-            <parent link="base_link"/>
-            <child link="battery"/>
-            <origin xyz="-0.25 0. 0." rpy="0 0 0"/>
+            <parent link="base_link" />
+            <child link="battery" />
+            <origin xyz="-0.25 0. 0." rpy="0 0 0" />
         </joint>
     </xacro:macro>

File: robot_description/src/description/robot_parts/caster_wheel.xacro (robot description, xacro)
@@ -22,22 +22,22 @@
             <visual>
                 <geometry>
-                    <sphere radius="${(wheel_radius+wheel_zoff-(base_height/2))}"/>
+                    <sphere radius="${(wheel_radius+wheel_zoff-(base_height/2))}" />
                 </geometry>
                 <material name="Cyan">
-                    <color rgba="0 1.0 1.0 1.0"/>
+                    <color rgba="0 1.0 1.0 1.0" />
                 </material>
             </visual>
             <collision>
-                <origin xyz="0 0 0" rpy="0 0 0"/>
+                <origin xyz="0 0 0" rpy="0 0 0" />
                 <geometry>
-                    <sphere radius="${(wheel_radius+wheel_zoff-(base_height/2))}"/>
+                    <sphere radius="${(wheel_radius+wheel_zoff-(base_height/2))}" />
                 </geometry>
             </collision>
-            <xacro:sphere_inertia m="0.5" r="${(wheel_radius+wheel_zoff-(base_height/2))}"/>
+            <xacro:sphere_inertia m="0.5" r="${(wheel_radius+wheel_zoff-(base_height/2))}" />
         </link>
         <joint name="caster_joint" type="fixed">
-            <parent link="base_link"/>
-            <child link="front_caster"/>
-            <origin xyz="${caster_xoff} 0.0 ${-(base_height/2)}" rpy="0 0 0"/>
+            <parent link="base_link" />
+            <child link="front_caster" />
+            <origin xyz="${caster_xoff} 0.0 ${-(base_height/2)}" rpy="0 0 0" />
         </joint>
     </xacro:macro>

File: robot_description/src/description/robot_parts/collector/collector.xacro (robot description, xacro)
@@ -2,25 +2,27 @@
 <robot name="collector"
     xmlns:xacro="http://ros.org/wiki/xacro">
-    <xacro:include filename="$(find robot_description)/src/description/robot_parts/collector/segment.xacro" />
+    <xacro:include
+        filename="$(find robot_description)/src/description/robot_parts/collector/segment.xacro" />
     <xacro:macro name="collector">
-        <!-- <xacro:segment name="segment_central" x="0.7" y="0.05" z="0.2" joint_parent="base_link" joint_origin_xyz="0.25 0.0 0" joint_origin_rpy="0 0 ${0.5 * pi}"/> -->
+        <!-- <xacro:segment name="segment_central" x="0.7" y="0.05" z="0.2" joint_parent="base_link"
+        joint_origin_xyz="0.25 0.0 0" joint_origin_rpy="0 0 ${0.5 * pi}"/> -->
         <gazebo reference="segment_central">
             <visual>
-            <material>
-            <ambient>1. 0.3 0.3 1.0</ambient>
-            <diffuse>1. 0.3 0.3 1.0</diffuse>
-            <specular>1. 0.3 0.3 1.0</specular>
-            <emissive>1. 0.3 0.3 1.0</emissive>
-            </material>
+                <material>
+                    <ambient>1. 0.3 0.3 1.0</ambient>
+                    <diffuse>1. 0.3 0.3 1.0</diffuse>
+                    <specular>1. 0.3 0.3 1.0</specular>
+                    <emissive>1. 0.3 0.3 1.0</emissive>
+                </material>
             </visual>
         </gazebo>
         <link name="segment_central">
             <visual>
-            <geometry>
-                <box size="0.7 0.05 0.2"/>
-            </geometry>
-            <material name="Brown">
-                <color rgba="0.30 0.15 0.0 1.0"/>
-            </material>
+                <geometry>
+                    <box size="0.7 0.05 0.2" />
+                </geometry>
+                <material name="Brown">
+                    <color rgba="0.30 0.15 0.0 1.0" />
+                </material>
             </visual>
             <!-- <collision>
@@ -30,17 +32,17 @@
             </geometry>
             </collision> -->
-            <xacro:box_inertia m="0.1" w="0.7" d="0.05" h="0.2"/>
+            <xacro:box_inertia m="0.1" w="0.7" d="0.05" h="0.2" />
         </link>
         <joint name="segment_central_joint" type="revolute">
-            <axis xyz="1 0 0"/>
-            <origin xyz="0.25 0.0 0" rpy="-1.5 0 ${-0.5 * pi}"/>
-            <parent link="base_link"/>
-            <child link="segment_central"/>
-            <limit effort="1000.0" lower="-0.15" upper="0.15" velocity="30"/>
+            <axis xyz="1 0 0" />
+            <origin xyz="0.25 0.0 0" rpy="-1.5 0 ${-0.5 * pi}" />
+            <parent link="base_link" />
+            <child link="segment_central" />
+            <limit effort="1000.0" lower="-0.15" upper="0.15" velocity="30" />
             <!-- <dynamics damping="0.0" friction="0.0"/> -->
         </joint>
         <ros2_control name="GazeboSystem" type="system">
             <hardware>
-            <plugin>gazebo_ros2_control/GazeboSystem</plugin>
+                <plugin>gazebo_ros2_control/GazeboSystem</plugin>
             </hardware>
             <joint name="segment_central_joint">
@@ -49,22 +51,32 @@
                     <param name="max">0.10</param>
                 </command_interface>
-                <state_interface name="position"/>
-                <state_interface name="velocity"/>
-                <state_interface name="effort"/>
+                <state_interface name="position" />
+                <state_interface name="velocity" />
+                <state_interface name="effort" />
             </joint>
         </ros2_control>
         <gazebo>
             <plugin filename="libgazebo_ros2_control.so" name="gazebo_ros2_control">
-            <parameters>$(find robot_description)/config/gripper_controller.yaml</parameters>
+                <parameters>$(find robot_description)/config/gripper_controller.yaml</parameters>
             </plugin>
         </gazebo>
-        <xacro:segment name="segment_d1" x="0.3" y="0.05" z="0.2" joint_parent="segment_central" joint_origin_xyz="-.25 -.32 0" joint_origin_rpy="0 0 ${0.16 * pi}"/>
-        <xacro:segment name="segment_d2" x="0.3" y="0.05" z="0.2" joint_parent="segment_d1" joint_origin_xyz="-0.30 -0.07 0" joint_origin_rpy="0 0 ${0.16 * pi}"/>
-        <xacro:segment name="segment_d3" x="0.3" y="0.05" z="0.2" joint_parent="segment_d2" joint_origin_xyz="-0.15 -0.1 0" joint_origin_rpy="0 0 ${-0.32* pi}"/>
-        <xacro:segment name="segment_g1" x="0.3" y="0.05" z="0.2" joint_parent="segment_central" joint_origin_xyz="0.25 -0.32 0" joint_origin_rpy="0 0 ${-0.16* pi}"/>
-        <xacro:segment name="segment_g2" x="0.3" y="0.05" z="0.2" joint_parent="segment_g1" joint_origin_xyz="0.30 -0.07 0" joint_origin_rpy="0 0 ${-0.16* pi}"/>
-        <xacro:segment name="segment_g3" x="0.3" y="0.05" z="0.2" joint_parent="segment_g2" joint_origin_xyz="0.15 -0.1 0" joint_origin_rpy="0 0 ${0.32* pi}"/>
-        <xacro:segment name="segment_triangled" x="0.3" y="0.05" z="0.2"  joint_parent="segment_central" joint_origin_xyz="-0.25 -0.12 0" joint_origin_rpy="0 0 ${-0.25* pi}"/>
-        <xacro:segment name="segment_triangleg" x="0.3" y="0.05" z="0.2"  joint_parent="segment_central" joint_origin_xyz="0.25 -0.12 0" joint_origin_rpy="0 0 ${0.25* pi}"/>
+        <xacro:segment name="segment_d1" x="0.3" y="0.05" z="0.2" joint_parent="segment_central"
+            joint_origin_xyz="-.25 -.32 0" joint_origin_rpy="0 0 ${0.16 * pi}" />
+        <xacro:segment name="segment_d2" x="0.3" y="0.05" z="0.2" joint_parent="segment_d1"
+            joint_origin_xyz="-0.30 -0.07 0" joint_origin_rpy="0 0 ${0.16 * pi}" />
+        <xacro:segment name="segment_d3" x="0.3" y="0.05" z="0.2" joint_parent="segment_d2"
+            joint_origin_xyz="-0.15 -0.1 0" joint_origin_rpy="0 0 ${-0.32* pi}" />
+        <xacro:segment name="segment_g1" x="0.3" y="0.05" z="0.2" joint_parent="segment_central"
+            joint_origin_xyz="0.25 -0.32 0" joint_origin_rpy="0 0 ${-0.16* pi}" />
+        <xacro:segment name="segment_g2" x="0.3" y="0.05" z="0.2" joint_parent="segment_g1"
+            joint_origin_xyz="0.30 -0.07 0" joint_origin_rpy="0 0 ${-0.16* pi}" />
+        <xacro:segment name="segment_g3" x="0.3" y="0.05" z="0.2" joint_parent="segment_g2"
+            joint_origin_xyz="0.15 -0.1 0" joint_origin_rpy="0 0 ${0.32* pi}" />
+        <xacro:segment name="segment_triangled" x="0.3" y="0.05" z="0.2"
+            joint_parent="segment_central" joint_origin_xyz="-0.25 -0.12 0"
+            joint_origin_rpy="0 0 ${-0.25* pi}" />
+        <xacro:segment name="segment_triangleg" x="0.3" y="0.05" z="0.2"
+            joint_parent="segment_central" joint_origin_xyz="0.25 -0.12 0"
+            joint_origin_rpy="0 0 ${0.25* pi}" />
     </xacro:macro>
 </robot>

File: robot_description/src/description/robot_parts/collector/segment.xacro (robot description, xacro)
@@ -16,8 +16,8 @@
             <visual>
                 <geometry>
-                    <box size="${x} ${y} ${z}"/>
+                    <box size="${x} ${y} ${z}" />
                 </geometry>
                 <material name="Brown">
-                    <color rgba="0.30 0.15 0.0 1.0"/>
+                    <color rgba="0.30 0.15 0.0 1.0" />
                 </material>
             </visual>
@@ -28,10 +28,10 @@
                 </geometry>
             </collision> -->
-            <xacro:box_inertia m="0.1" w="${x}" d="${y}" h="${z}"/>
+            <xacro:box_inertia m="0.1" w="${x}" d="${y}" h="${z}" />
         </link>
         <joint name="${name}_joint" type="fixed">
-            <parent link="${joint_parent}"/>
-            <child link="${name}"/>
-            <origin xyz="${joint_origin_xyz}" rpy="${joint_origin_rpy}"/>
+            <parent link="${joint_parent}" />
+            <child link="${name}" />
+            <origin xyz="${joint_origin_xyz}" rpy="${joint_origin_rpy}" />
         </joint>
     </xacro:macro>

File: robot_description/src/description/robot_parts/property.xacro (robot description, xacro)
@@ -3,25 +3,26 @@
     xmlns:xacro="http://ros.org/wiki/xacro">
     <!-- Define robot constants -->
-    <xacro:property name="base_width" value="0.31"/>
-    <xacro:property name="base_length" value="0.42"/>
-    <xacro:property name="base_height" value="0.18"/>
-    <xacro:property name="wheel_radius" value="0.10"/>
-    <xacro:property name="wheel_width" value="0.04"/>
-    <xacro:property name="wheel_ygap" value="0.025"/>
-    <xacro:property name="wheel_zoff" value="0.05"/>
-    <xacro:property name="wheel_xoff" value="0.12"/>
-    <xacro:property name="caster_xoff" value="0.14"/>
+    <xacro:property name="base_width" value="0.31" />
+    <xacro:property name="base_length" value="0.42" />
+    <xacro:property name="base_height" value="0.18" />
+    <xacro:property name="wheel_radius" value="0.10" />
+    <xacro:property name="wheel_width" value="0.04" />
+    <xacro:property name="wheel_ygap" value="0.025" />
+    <xacro:property name="wheel_zoff" value="0.05" />
+    <xacro:property name="wheel_xoff" value="0.12" />
+    <xacro:property name="caster_xoff" value="0.14" />
     <material name="corps">
-        <color rgba="0.3 1. 0.3 1.0"/>
+        <color rgba="0.3 1. 0.3 1.0" />
     </material>
     <material name="reste">
-        <color rgba="1. 0.3 0.3 1.0"/>
+        <color rgba="1. 0.3 0.3 1.0" />
     </material>
     <!-- Define some commonly used intertial properties  -->
     <xacro:macro name="box_inertia" params="m w h d">
         <inertial>
-            <origin xyz="0 0 0" rpy="${pi/2} 0 ${pi/2}"/>
-            <mass value="${m}"/>
-            <inertia ixx="${(m/12) * (h*h + d*d)}" ixy="0.0" ixz="0.0" iyy="${(m/12) * (w*w + d*d)}" iyz="0.0" izz="${(m/12) * (w*w + h*h)}"/>
+            <origin xyz="0 0 0" rpy="${pi/2} 0 ${pi/2}" />
+            <mass value="${m}" />
+            <inertia ixx="${(m/12) * (h*h + d*d)}" ixy="0.0" ixz="0.0" iyy="${(m/12) * (w*w + d*d)}"
+                iyz="0.0" izz="${(m/12) * (w*w + h*h)}" />
         </inertial>
     </xacro:macro>
@@ -29,12 +30,14 @@
         <inertial>
             <origin xyz="0 0 0" rpy="${pi/2} 0 0" />
-            <mass value="${m}"/>
-            <inertia ixx="${(m/12) * (3*r*r + h*h)}" ixy = "0" ixz = "0" iyy="${(m/12) * (3*r*r + h*h)}" iyz = "0" izz="${(m/2) * (r*r)}"/>
+            <mass value="${m}" />
+            <inertia ixx="${(m/12) * (3*r*r + h*h)}" ixy="0" ixz="0" iyy="${(m/12) * (3*r*r + h*h)}"
+                iyz="0" izz="${(m/2) * (r*r)}" />
         </inertial>
     </xacro:macro>
     <xacro:macro name="sphere_inertia" params="m r">
         <inertial>
-            <mass value="${m}"/>
-            <inertia ixx="${(2/5) * m * (r*r)}" ixy="0.0" ixz="0.0" iyy="${(2/5) * m * (r*r)}" iyz="0.0" izz="${(2/5) * m * (r*r)}"/>
+            <mass value="${m}" />
+            <inertia ixx="${(2/5) * m * (r*r)}" ixy="0.0" ixz="0.0" iyy="${(2/5) * m * (r*r)}"
+                iyz="0.0" izz="${(2/5) * m * (r*r)}" />
         </inertial>
     </xacro:macro>

File: robot_description/src/description/robot_parts/wheels.xacro (robot description, xacro)
@@ -27,25 +27,27 @@
             <link name="${prefix}_link">
                 <visual>
-                    <origin xyz="0 0 0" rpy="${pi/2} 0 0"/>
+                    <origin xyz="0 0 0" rpy="${pi/2} 0 0" />
                     <geometry>
-                        <cylinder radius="${wheel_radius}" length="${wheel_width}"/>
+                        <cylinder radius="${wheel_radius}" length="${wheel_width}" />
                     </geometry>
                     <material name="Gray">
-                        <color rgba="0.5 0.5 0.5 1.0"/>
+                        <color rgba="0.5 0.5 0.5 1.0" />
                     </material>
                 </visual>
                 <collision>
-                    <origin xyz="0 0 0" rpy="${pi/2} 0 0"/>
+                    <origin xyz="0 0 0" rpy="${pi/2} 0 0" />
                     <geometry>
-                        <cylinder radius="${wheel_radius}" length="${wheel_width}"/>
+                        <cylinder radius="${wheel_radius}" length="${wheel_width}" />
                     </geometry>
                 </collision>
-                <xacro:cylinder_inertia m="0.5" r="${wheel_radius}" h="${wheel_width}"/>
+                <xacro:cylinder_inertia m="0.5" r="${wheel_radius}" h="${wheel_width}" />
             </link>
             <joint name="${prefix}_joint" type="continuous">
-                <parent link="base_link"/>
-                <child link="${prefix}_link"/>
-                <origin xyz="${x_reflect*wheel_xoff} ${y_reflect*(base_width/2+wheel_ygap)} ${-wheel_zoff}" rpy="0 0 0"/>
-                <axis xyz="0 1 0"/>
+                <parent link="base_link" />
+                <child link="${prefix}_link" />
+                <origin
+                    xyz="${x_reflect*wheel_xoff} ${y_reflect*(base_width/2+wheel_ygap)} ${-wheel_zoff}"
+                    rpy="0 0 0" />
+                <axis xyz="0 1 0" />
             </joint>
         </xacro:macro>
