Commit message: Work: Pince complète

File: robot_description/src/description/robot_parts/base.xacro (robot description, xacro)
@@ -16,5 +16,6 @@
         <link name="base_link">
             <visual>
-                <origin xyz="-0.2 -0.15 0" rpy="${pi/2} 0 0" />
+                <!-- <origin xyz="-0.2 -0.15 0" rpy="${pi/2} 0 0" /> -->
+                <origin xyz="-0.2 -0.15 -0.06" rpy="${pi/2} 0 0" />
                 <geometry>
                     <mesh filename="$(find robot_description)/src/description/robot_parts/meshes/chassis_is.dae" scale="0.001 0.001 0.001"/>

File: robot_description/src/description/robot_parts/collector2/collector.xacro (robot description, xacro)
@@ -17,8 +17,8 @@
         <link name="segment_central">
             <visual>
-            <origin xyz="-0.35 0 0" rpy="0 0 0"/>
+            <origin xyz="-0.25 0 0" rpy="0 0 0"/>
             <geometry>
                 <!-- <box size="0.7 0.05 0.2"/> -->
-                <box size="0.7 0.01 0.2"/>
+                <box size="0.5 0.01 0.2"/>
             </geometry>
             <material name="Brown">
@@ -32,13 +32,13 @@
             </geometry>
             </collision> -->
-            <xacro:box_inertia m="0.01" w="0.7" d="0.05" h="0.2"/>
+            <xacro:box_inertia m="0.00001" w="0.7" d="0.05" h="0.2"/>
         </link>
         <joint name="segment_central_joint" type="revolute">
             <axis xyz="0 1 0"/>
             <!-- <origin xyz="0.25 -0.23 0" rpy="-1.5 0 ${-0.5 * pi}"/> -->
-            <origin xyz="0 -0.23 0" rpy="${0 * pi} ${0 * pi} ${0 * pi}"/>
+            <origin xyz="0.1 -0.23 0" rpy="${0 * pi} ${(-1/20) * pi} ${0 * pi}"/>
             <parent link="base_link"/>
             <child link="segment_central"/>
-            <limit effort="1000.0" lower="${-1 * pi}" upper="${1 * pi}" velocity="30"/>
+            <limit effort="1.0" lower="${(1/20) * pi}" upper="${(1+1/20) * pi}" velocity="30"/>
             <!-- <dynamics damping="0.0" friction="0.0"/> -->
         </joint>
@@ -62,6 +62,7 @@
             </plugin>
         </gazebo>
-        <!-- <xacro:segment name="segment_d1" x="0.3" y="0.05" z="0.2" joint_parent="segment_central" joint_origin_xyz="-.25 -.32 0" joint_origin_rpy="0 0 ${0.16 * pi}"/>
-        <xacro:segment name="segment_d2" x="0.3" y="0.05" z="0.2" joint_parent="segment_d1" joint_origin_xyz="-0.30 -0.07 0" joint_origin_rpy="0 0 ${0.16 * pi}"/>
+        <xacro:segment name="segment_g" x="0.7" y="0.01" z="0.2" joint_parent="segment_central" joint_origin_xyz="-0.35 0.46 0" joint_origin_rpy="0 ${0* pi} ${0 * pi}"/>
+        <!-- <xacro:segment name="fermeture_d" x="0.2" y="0.01" z="0.2" joint_parent="segment_central" joint_origin_xyz="-0.35 0 0" joint_origin_rpy="${0* pi} ${0* pi} ${(1/6) * pi}"/> -->
+        <!-- <xacro:segment name="segment_d2" x="0.3" y="0.05" z="0.2" joint_parent="segment_d1" joint_origin_xyz="-0.30 -0.07 0" joint_origin_rpy="0 0 ${0.16 * pi}"/>
         <xacro:segment name="segment_d3" x="0.3" y="0.05" z="0.2" joint_parent="segment_d2" joint_origin_xyz="-0.15 -0.1 0" joint_origin_rpy="0 0 ${-0.32* pi}"/>
         <xacro:segment name="segment_g1" x="0.3" y="0.05" z="0.2" joint_parent="segment_central" joint_origin_xyz="0.25 -0.32 0" joint_origin_rpy="0 0 ${-0.16* pi}"/>

File: robot_description/src/description/robot_parts/collector2/segment.xacro (robot description, xacro)
@@ -28,5 +28,5 @@
                 </geometry>
             </collision> -->
-            <xacro:box_inertia m="0.1" w="${x}" d="${y}" h="${z}"/>
+            <xacro:box_inertia m="0.00001" w="${x}" d="${y}" h="${z}"/>
         </link>
         <joint name="${name}_joint" type="fixed">

File: robot_description/src/description/robot_parts/property.xacro (robot description, xacro)
@@ -6,5 +6,5 @@
     <xacro:property name="base_length" value="0.42"/>
     <xacro:property name="base_height" value="0.18"/>
-    <xacro:property name="wheel_radius" value="0.10"/>
+    <xacro:property name="wheel_radius" value="0.07"/>
     <xacro:property name="wheel_width" value="0.04"/>
     <xacro:property name="wheel_ygap" value="0.025"/>

Commit message: traitement image pince corrige

File: robot_description/src/description/robot_parts/base.xacro (robot description, xacro)
@@ -34,4 +34,35 @@
             <xacro:box_inertia m="15" w="${base_width}" d="${base_length}" h="${base_height}" />
         </link>
+        <!-- <gazebo reference="cap">
+            <visual>
+                <material>
+                    <ambient>1. 0.3 0.3 1.0</ambient>
+                    <diffuse>1. 0.3 0.3 1.0</diffuse>
+                    <specular>1. 0.3 0.3 1.0</specular>
+                    <emissive>1. 0.3 0.3 1.0</emissive>
+                </material>
+            </visual>
+        </gazebo>
+        <link name="cap">
+            <visual>
+                <geometry>
+                    <box size="0.4 0.40 0.01" />
+                </geometry>
+                <material name="Brown">
+                    <color rgba="0.35 0.15 0.0 1.0" />
+                </material>
+            </visual>
+            <collision>
+                <geometry>
+                    <box size="0.4 0.40 0.01" />
+                </geometry>
+            </collision>
+            <xacro:box_inertia m="0.00001" w="0.7" d="0.05" h="0.2" />
+        </link>
+        <joint name="cap_joint" type="fixed">
+            <origin xyz="0.25 0 0.1" rpy="0 0 0" />
+            <parent link="base_link" />
+            <child link="cap" />
+        </joint> -->
         <!-- Robot Footprint -->
         <link name="base_footprint">

File: robot_description/src/description/robot_parts/collector2/collector.xacro (robot description, xacro)
@@ -120,15 +120,15 @@
                 <geometry>
                     <!-- <box size="0.7 0.05 0.2"/> -->
-                    <box size="0.2 0.01 0.2" />
-                </geometry>
-                <material name="Brown">
-                    <color rgba="0.30 0.15 0.0 1.0" />
-                </material>
-            </visual>
-            <collision>
-                <origin xyz="-0.15 0 0" rpy="0 0 0" />
-                <geometry>
-                    <!-- <box size="0.7 0.05 0.2"/> -->
-                    <box size="0.2 0.01 0.2" />
+                    <box size="0.15 0.01 0.2" />
+                </geometry>
+                <material name="Brown">
+                    <color rgba="0.30 0.15 0.0 1.0" />
+                </material>
+            </visual>
+            <collision>
+                <!-- <origin xyz="-0.15 0 0" rpy="0 0 0" /> -->
+                <geometry>
+                    <!-- <box size="0.7 0.05 0.2"/> -->
+                    <box size="0.15 0.01 0.2" />
                 </geometry>
             </collision>
@@ -159,15 +159,15 @@
                 <geometry>
                     <!-- <box size="0.7 0.05 0.2"/> -->
-                    <box size="0.2 0.01 0.2" />
-                </geometry>
-                <material name="Brown">
-                    <color rgba="0.30 0.15 0.0 1.0" />
-                </material>
-            </visual>
-            <collision>
-                <origin xyz="-0.15 0 0" rpy="0 0 0" />
-                <geometry>
-                    <!-- <box size="0.7 0.05 0.2"/> -->
-                    <box size="0.2 0.01 0.2" />
+                    <box size="0.15 0.01 0.2" />
+                </geometry>
+                <material name="Brown">
+                    <color rgba="0.30 0.15 0.0 1.0" />
+                </material>
+            </visual>
+            <collision>
+                <!-- <origin xyz="-0.15 0 0" rpy="0 0 0" /> -->
+                <geometry>
+                    <!-- <box size="0.7 0.05 0.2"/> -->
+                    <box size="0.15 0.01 0.2" />
                 </geometry>
             </collision>
