Commit message: Work: 1 pince, mauvaise axe de rotation

File: robot_description/src/description/robot_parts/collector2/collector.xacro (robot description, xacro)
@@ -34,10 +34,10 @@
         </link>
         <joint name="segment_central_joint" type="revolute">
-            <axis xyz="1 0 0"/>
+            <axis xyz="0 1 0"/>
             <!-- <origin xyz="0.25 -0.23 0" rpy="-1.5 0 ${-0.5 * pi}"/> -->
             <origin xyz="-0.5 -0.23 0" rpy="${0 * pi} ${0 * pi} ${0 * pi}"/>
             <parent link="base_link"/>
             <child link="segment_central"/>
-            <limit effort="1000.0" lower="-0.15" upper="0.15" velocity="30"/>
+            <limit effort="1000.0" lower="${-1 * pi}" upper="${1 * pi}" velocity="30"/>
             <!-- <dynamics damping="0.0" friction="0.0"/> -->
         </joint>

Commit message: Done: 1pince articulé

File: robot_description/src/description/robot_parts/collector2/collector.xacro (robot description, xacro)
@@ -17,4 +17,5 @@
         <link name="segment_central">
             <visual>
+            <origin xyz="-0.35 0 0" rpy="0 0 0"/>
             <geometry>
                 <!-- <box size="0.7 0.05 0.2"/> -->
@@ -31,10 +32,10 @@
             </geometry>
             </collision> -->
-            <xacro:box_inertia m="0.1" w="0.7" d="0.05" h="0.2"/>
+            <xacro:box_inertia m="0.01" w="0.7" d="0.05" h="0.2"/>
         </link>
         <joint name="segment_central_joint" type="revolute">
             <axis xyz="0 1 0"/>
             <!-- <origin xyz="0.25 -0.23 0" rpy="-1.5 0 ${-0.5 * pi}"/> -->
-            <origin xyz="-0.5 -0.23 0" rpy="${0 * pi} ${0 * pi} ${0 * pi}"/>
+            <origin xyz="0 -0.23 0" rpy="${0 * pi} ${0 * pi} ${0 * pi}"/>
             <parent link="base_link"/>
             <child link="segment_central"/>

Commit message: Pince Ok pas nickel

File: robot_description/src/description/robot_parts/collector2/collector.xacro (robot description, xacro)
@@ -17,8 +17,8 @@
         <link name="segment_central">
             <visual>
-            <origin xyz="-0.25 0 0" rpy="0 0 0"/>
+            <origin xyz="-0.15 0 0" rpy="0 0 0"/>
             <geometry>
                 <!-- <box size="0.7 0.05 0.2"/> -->
-                <box size="0.5 0.01 0.2"/>
+                <box size="0.3 0.01 0.2"/>
             </geometry>
             <material name="Brown">
@@ -26,10 +26,11 @@
             </material>
             </visual>
-            <!-- <collision>
-            <origin xyz="0 0 0" rpy="0 0 0"/>
-            <geometry>0 0.0 0.0 1.0
-                <box size="0.7 0.05 0.2"/>
+            <collision>
+            <origin xyz="-0.15 0 0" rpy="0 0 0"/>
+            <geometry>
+                <!-- <box size="0.7 0.05 0.2"/> -->
+                <box size="0.3 0.01 0.2"/>
             </geometry>
-            </collision> -->
+            </collision>
             <xacro:box_inertia m="0.00001" w="0.7" d="0.05" h="0.2"/>
         </link>
@@ -62,6 +63,124 @@
             </plugin>
         </gazebo>
-        <xacro:segment name="segment_g" x="0.7" y="0.01" z="0.2" joint_parent="segment_central" joint_origin_xyz="-0.35 0.46 0" joint_origin_rpy="0 ${0* pi} ${0 * pi}"/>
-        <!-- <xacro:segment name="fermeture_d" x="0.2" y="0.01" z="0.2" joint_parent="segment_central" joint_origin_xyz="-0.35 0 0" joint_origin_rpy="${0* pi} ${0* pi} ${(1/6) * pi}"/> -->
+        <!--  -->
+        <gazebo reference="segment_g">
+            <visual>
+            <material>
+            <ambient>1. 0.3 0.3 1.0</ambient>
+            <diffuse>1. 0.3 0.3 1.0</diffuse>
+            <specular>1. 0.3 0.3 1.0</specular>
+            <emissive>1. 0.3 0.3 1.0</emissive>
+            </material>
+            </visual>
+        </gazebo>
+        <link name="segment_g">
+            <visual>
+            <!-- <origin xyz="-0.15 0 0" rpy="0 0 0"/> -->
+            <geometry>
+                <!-- <box size="0.7 0.05 0.2"/> -->
+                <box size="0.3 0.01 0.2"/>
+            </geometry>
+            <material name="Brown">
+                <color rgba="0.30 0.15 0.0 1.0"/>
+            </material>
+            </visual>
+            <collision>
+            <origin xyz="-0.15 0 0" rpy="0 0 0"/>
+            <geometry>
+                <!-- <box size="0.7 0.05 0.2"/> -->
+                <box size="0.3 0.01 0.2"/>
+            </geometry>
+            </collision>
+            <xacro:box_inertia m="0.00001" w="0.7" d="0.05" h="0.2"/>
+        </link>
+        <joint name="segment_g_joint" type="fixed">
+            <!-- <axis xyz="0 1 0"/> -->
+            <!-- <origin xyz="0.25 -0.23 0" rpy="-1.5 0 ${-0.5 * pi}"/> -->
+            <origin xyz="-0.15 0.46 0" rpy="${0 * pi} ${(0) * pi} ${0 * pi}"/>
+            <parent link="segment_central"/>
+            <child link="segment_g"/>
+            <!-- <dynamics damping="0.0" friction="0.0"/> -->
+        </joint>
+        <!--  -->
+        <gazebo reference="pince_d">
+            <visual>
+            <material>
+            <ambient>1. 0.3 0.3 1.0</ambient>
+            <diffuse>1. 0.3 0.3 1.0</diffuse>
+            <specular>1. 0.3 0.3 1.0</specular>
+            <emissive>1. 0.3 0.3 1.0</emissive>
+            </material>
+            </visual>
+        </gazebo>
+        <link name="pince_d">
+            <visual>
+            <!-- <origin xyz="-0.15 0 0" rpy="0 0 0"/> -->
+            <geometry>
+                <!-- <box size="0.7 0.05 0.2"/> -->
+                <box size="0.2 0.01 0.2"/>
+            </geometry>
+            <material name="Brown">
+                <color rgba="0.30 0.15 0.0 1.0"/>
+            </material>
+            </visual>
+            <collision>
+            <origin xyz="-0.15 0 0" rpy="0 0 0"/>
+            <geometry>
+                <!-- <box size="0.7 0.05 0.2"/> -->
+                <box size="0.2 0.01 0.2"/>
+            </geometry>
+            </collision>
+            <xacro:box_inertia m="0.00001" w="0.7" d="0.05" h="0.2"/>
+        </link>
+        <joint name="pince_d_joint" type="fixed">
+            <!-- <axis xyz="0 1 0"/> -->
+            <!-- <origin xyz="0.25 -0.23 0" rpy="-1.5 0 ${-0.5 * pi}"/> -->
+            <origin xyz="-0.4 0.05 0" rpy="${0* pi} ${0* pi} ${(-1/4) * pi}"/>
+            <parent link="segment_central"/>
+            <child link="pince_d"/>
+            <!-- <dynamics damping="0.0" friction="0.0"/> -->
+        </joint>
+        <!--  -->
+        <gazebo reference="pince_g">
+            <visual>
+            <material>
+            <ambient>1. 0.3 0.3 1.0</ambient>
+            <diffuse>1. 0.3 0.3 1.0</diffuse>
+            <specular>1. 0.3 0.3 1.0</specular>
+            <emissive>1. 0.3 0.3 1.0</emissive>
+            </material>
+            </visual>
+        </gazebo>
+        <link name="pince_g">
+            <visual>
+            <!-- <origin xyz="-0.15 0 0" rpy="0 0 0"/> -->
+            <geometry>
+                <!-- <box size="0.7 0.05 0.2"/> -->
+                <box size="0.2 0.01 0.2"/>
+            </geometry>
+            <material name="Brown">
+                <color rgba="0.30 0.15 0.0 1.0"/>
+            </material>
+            </visual>
+            <collision>
+            <origin xyz="-0.15 0 0" rpy="0 0 0"/>
+            <geometry>
+                <!-- <box size="0.7 0.05 0.2"/> -->
+                <box size="0.2 0.01 0.2"/>
+            </geometry>
+            </collision>
+            <xacro:box_inertia m="0.00001" w="0.7" d="0.05" h="0.2"/>
+        </link>
+        <joint name="pince_g_joint" type="fixed">
+            <!-- <axis xyz="0 1 0"/> -->
+            <!-- <origin xyz="0.25 -0.23 0" rpy="-1.5 0 ${-0.5 * pi}"/> -->
+            <origin xyz="-0.4 0.4 0" rpy="${0* pi} ${0* pi} ${(1/4) * pi}"/>
+            <parent link="segment_central"/>
+            <child link="pince_g"/>
+            <!-- <dynamics damping="0.0" friction="0.0"/> -->
+        </joint>
+<!--
+        <xacro:segment name="segment_g" x="0.3" y="0.01" z="0.2" joint_parent="segment_central" joint_origin_xyz="-0.25 0.46 0" joint_origin_rpy="0 ${0* pi} ${0 * pi}"/>
+        <xacro:segment name="fermeture_d" x="0.2" y="0.01" z="0.2" joint_parent="segment_central" joint_origin_xyz="-0.4 0.05 0" joint_origin_rpy="${0* pi} ${0* pi} ${(-1/4) * pi}"/> -->
         <!-- <xacro:segment name="segment_d2" x="0.3" y="0.05" z="0.2" joint_parent="segment_d1" joint_origin_xyz="-0.30 -0.07 0" joint_origin_rpy="0 0 ${0.16 * pi}"/>
         <xacro:segment name="segment_d3" x="0.3" y="0.05" z="0.2" joint_parent="segment_d2" joint_origin_xyz="-0.15 -0.1 0" joint_origin_rpy="0 0 ${-0.32* pi}"/>

File: robot_description/src/description/robot_parts/collector2/segment.xacro (robot description, xacro)
@@ -22,10 +22,10 @@
                 </material>
             </visual>
-            <!-- <collision>
+            <collision>
                 <origin xyz="0 0 0" rpy="0 0 0"/>
-                <geometry>0 0.0 0.0 1.0
+                <geometry>
                     <box size="${x} ${y} ${z}"/>
                 </geometry>
-            </collision> -->
+            </collision>
             <xacro:box_inertia m="0.00001" w="${x}" d="${y}" h="${z}"/>
         </link>
