Commit message: pep8 sur collector

File: robot_description/src/description/robot_parts/collector2/collector.xacro (robot description, xacro)
@@ -2,49 +2,51 @@
 <robot name="collector"
     xmlns:xacro="http://ros.org/wiki/xacro">
-    <xacro:include filename="$(find robot_description)/src/description/robot_parts/collector/segment.xacro" />
+    <xacro:include
+        filename="$(find robot_description)/src/description/robot_parts/collector/segment.xacro" />
     <xacro:macro name="collector">
-        <!-- <xacro:segment name="segment_central" x="0.7" y="0.05" z="0.2" joint_parent="base_link" joint_origin_xyz="0.25 0.0 0" joint_origin_rpy="0 0 ${0.5 * pi}"/> -->
+        <!-- <xacro:segment name="segment_central" x="0.7" y="0.05" z="0.2" joint_parent="base_link"
+        joint_origin_xyz="0.25 0.0 0" joint_origin_rpy="0 0 ${0.5 * pi}"/> -->
         <gazebo reference="segment_central">
             <visual>
-            <material>
-            <ambient>1. 0.3 0.3 1.0</ambient>
-            <diffuse>1. 0.3 0.3 1.0</diffuse>
-            <specular>1. 0.3 0.3 1.0</specular>
-            <emissive>1. 0.3 0.3 1.0</emissive>
-            </material>
+                <material>
+                    <ambient>1. 0.3 0.3 1.0</ambient>
+                    <diffuse>1. 0.3 0.3 1.0</diffuse>
+                    <specular>1. 0.3 0.3 1.0</specular>
+                    <emissive>1. 0.3 0.3 1.0</emissive>
+                </material>
             </visual>
         </gazebo>
         <link name="segment_central">
             <visual>
-            <origin xyz="-0.15 0 0" rpy="0 0 0"/>
-            <geometry>
-                <!-- <box size="0.7 0.05 0.2"/> -->
-                <box size="0.3 0.01 0.2"/>
-            </geometry>
-            <material name="Brown">
-                <color rgba="0.30 0.15 0.0 1.0"/>
-            </material>
-            </visual>
-            <collision>
-            <origin xyz="-0.15 0 0" rpy="0 0 0"/>
-            <geometry>
-                <!-- <box size="0.7 0.05 0.2"/> -->
-                <box size="0.3 0.01 0.2"/>
-            </geometry>
-            </collision>
-            <xacro:box_inertia m="0.00001" w="0.7" d="0.05" h="0.2"/>
+                <origin xyz="-0.15 0 0" rpy="0 0 0" />
+                <geometry>
+                    <!-- <box size="0.7 0.05 0.2"/> -->
+                    <box size="0.3 0.01 0.2" />
+                </geometry>
+                <material name="Brown">
+                    <color rgba="0.30 0.15 0.0 1.0" />
+                </material>
+            </visual>
+            <collision>
+                <origin xyz="-0.15 0 0" rpy="0 0 0" />
+                <geometry>
+                    <!-- <box size="0.7 0.05 0.2"/> -->
+                    <box size="0.3 0.01 0.2" />
+                </geometry>
+            </collision>
+            <xacro:box_inertia m="0.00001" w="0.7" d="0.05" h="0.2" />
         </link>
         <joint name="segment_central_joint" type="revolute">
-            <axis xyz="0 1 0"/>
-            <!-- <origin xyz="0.25 -0.23 0" rpy="-1.5 0 ${-0.5 * pi}"/> -->
-            <origin xyz="0.1 -0.23 0" rpy="${0 * pi} ${(-1/20) * pi} ${0 * pi}"/>
-            <parent link="base_link"/>
-            <child link="segment_central"/>
-            <limit effort="1.0" lower="${(1/20) * pi}" upper="${(1+1/20) * pi}" velocity="30"/>
+            <axis xyz="0 1 0" />
+            <!-- <origin xyz="0.25 -0.23 0" rpy="-1.5 0 ${-0.5 * pi}"/> -->
+            <origin xyz="0.1 -0.23 0" rpy="${0 * pi} ${(-1/20) * pi} ${0 * pi}" />
+            <parent link="base_link" />
+            <child link="segment_central" />
+            <limit effort="1.0" lower="${(1/20) * pi}" upper="${(1+1/20) * pi}" velocity="30" />
             <!-- <dynamics damping="0.0" friction="0.0"/> -->
         </joint>
         <ros2_control name="GazeboSystem" type="system">
             <hardware>
-            <plugin>gazebo_ros2_control/GazeboSystem</plugin>
+                <plugin>gazebo_ros2_control/GazeboSystem</plugin>
             </hardware>
             <joint name="segment_central_joint">
@@ -53,12 +55,12 @@
                     <param name="max">0.10</param>
                 </command_interface>
-                <state_interface name="position"/>
-                <state_interface name="velocity"/>
-                <state_interface name="effort"/>
+                <state_interface name="position" />
+                <state_interface name="velocity" />
+                <state_interface name="effort" />
             </joint>
         </ros2_control>
         <gazebo>
             <plugin filename="libgazebo_ros2_control.so" name="gazebo_ros2_control">
-            <parameters>$(find robot_description)/config/gripper_controller.yaml</parameters>
+                <parameters>$(find robot_description)/config/gripper_controller.yaml</parameters>
             </plugin>
         </gazebo>
@@ -66,38 +68,38 @@
         <gazebo reference="segment_g">
             <visual>
-            <material>
-            <ambient>1. 0.3 0.3 1.0</ambient>
-            <diffuse>1. 0.3 0.3 1.0</diffuse>
-            <specular>1. 0.3 0.3 1.0</specular>
-            <emissive>1. 0.3 0.3 1.0</emissive>
-            </material>
+                <material>
+                    <ambient>1. 0.3 0.3 1.0</ambient>
+                    <diffuse>1. 0.3 0.3 1.0</diffuse>
+                    <specular>1. 0.3 0.3 1.0</specular>
+                    <emissive>1. 0.3 0.3 1.0</emissive>
+                </material>
             </visual>
         </gazebo>
         <link name="segment_g">
             <visual>
-            <!-- <origin xyz="-0.15 0 0" rpy="0 0 0"/> -->
-            <geometry>
-                <!-- <box size="0.7 0.05 0.2"/> -->
-                <box size="0.3 0.01 0.2"/>
-            </geometry>
-            <material name="Brown">
-                <color rgba="0.30 0.15 0.0 1.0"/>
-            </material>
-            </visual>
-            <collision>
-            <origin xyz="-0.15 0 0" rpy="0 0 0"/>
-            <geometry>
-                <!-- <box size="0.7 0.05 0.2"/> -->
-                <box size="0.3 0.01 0.2"/>
-            </geometry>
-            </collision>
-            <xacro:box_inertia m="0.00001" w="0.7" d="0.05" h="0.2"/>
+                <!-- <origin xyz="-0.15 0 0" rpy="0 0 0"/> -->
+                <geometry>
+                    <!-- <box size="0.7 0.05 0.2"/> -->
+                    <box size="0.3 0.01 0.2" />
+                </geometry>
+                <material name="Brown">
+                    <color rgba="0.30 0.15 0.0 1.0" />
+                </material>
+            </visual>
+            <collision>
+                <origin xyz="-0.15 0 0" rpy="0 0 0" />
+                <geometry>
+                    <!-- <box size="0.7 0.05 0.2"/> -->
+                    <box size="0.3 0.01 0.2" />
+                </geometry>
+            </collision>
+            <xacro:box_inertia m="0.00001" w="0.7" d="0.05" h="0.2" />
         </link>
         <joint name="segment_g_joint" type="fixed">
             <!-- <axis xyz="0 1 0"/> -->
             <!-- <origin xyz="0.25 -0.23 0" rpy="-1.5 0 ${-0.5 * pi}"/> -->
-            <origin xyz="-0.15 0.46 0" rpy="${0 * pi} ${(0) * pi} ${0 * pi}"/>
-            <parent link="segment_central"/>
-            <child link="segment_g"/>
+            <origin xyz="-0.15 0.46 0" rpy="${0 * pi} ${(0) * pi} ${0 * pi}" />
+            <parent link="segment_central" />
+            <child link="segment_g" />
             <!-- <dynamics damping="0.0" friction="0.0"/> -->
         </joint>
@@ -105,38 +107,38 @@
         <gazebo reference="pince_d">
             <visual>
-            <material>
-            <ambient>1. 0.3 0.3 1.0</ambient>
-            <diffuse>1. 0.3 0.3 1.0</diffuse>
-            <specular>1. 0.3 0.3 1.0</specular>
-            <emissive>1. 0.3 0.3 1.0</emissive>
-            </material>
+                <material>
+                    <ambient>1. 0.3 0.3 1.0</ambient>
+                    <diffuse>1. 0.3 0.3 1.0</diffuse>
+                    <specular>1. 0.3 0.3 1.0</specular>
+                    <emissive>1. 0.3 0.3 1.0</emissive>
+                </material>
             </visual>
         </gazebo>
         <link name="pince_d">
             <visual>
-            <!-- <origin xyz="-0.15 0 0" rpy="0 0 0"/> -->
-            <geometry>
-                <!-- <box size="0.7 0.05 0.2"/> -->
-                <box size="0.2 0.01 0.2"/>
-            </geometry>
-            <material name="Brown">
-                <color rgba="0.30 0.15 0.0 1.0"/>
-            </material>
-            </visual>
-            <collision>
-            <origin xyz="-0.15 0 0" rpy="0 0 0"/>
-            <geometry>
-                <!-- <box size="0.7 0.05 0.2"/> -->
-                <box size="0.2 0.01 0.2"/>
-            </geometry>
-            </collision>
-            <xacro:box_inertia m="0.00001" w="0.7" d="0.05" h="0.2"/>
+                <!-- <origin xyz="-0.15 0 0" rpy="0 0 0"/> -->
+                <geometry>
+                    <!-- <box size="0.7 0.05 0.2"/> -->
+                    <box size="0.2 0.01 0.2" />
+                </geometry>
+                <material name="Brown">
+                    <color rgba="0.30 0.15 0.0 1.0" />
+                </material>
+            </visual>
+            <collision>
+                <origin xyz="-0.15 0 0" rpy="0 0 0" />
+                <geometry>
+                    <!-- <box size="0.7 0.05 0.2"/> -->
+                    <box size="0.2 0.01 0.2" />
+                </geometry>
+            </collision>
+            <xacro:box_inertia m="0.00001" w="0.7" d="0.05" h="0.2" />
         </link>
         <joint name="pince_d_joint" type="fixed">
             <!-- <axis xyz="0 1 0"/> -->
             <!-- <origin xyz="0.25 -0.23 0" rpy="-1.5 0 ${-0.5 * pi}"/> -->
-            <origin xyz="-0.4 0.05 0" rpy="${0* pi} ${0* pi} ${(-1/4) * pi}"/>
-            <parent link="segment_central"/>
-            <child link="pince_d"/>
+            <origin xyz="-0.4 0.05 0" rpy="${0* pi} ${0* pi} ${(-1/4) * pi}" />
+            <parent link="segment_central" />
+            <child link="pince_d" />
             <!-- <dynamics damping="0.0" friction="0.0"/> -->
         </joint>
@@ -144,50 +146,59 @@
         <gazebo reference="pince_g">
             <visual>
-            <material>
-            <ambient>1. 0.3 0.3 1.0</ambient>
-            <diffuse>1. 0.3 0.3 1.0</diffuse>
-            <specular>1. 0.3 0.3 1.0</specular>
-            <emissive>1. 0.3 0.3 1.0</emissive>
-            </material>
+                <material>
+                    <ambient>1. 0.3 0.3 1.0</ambient>
+                    <diffuse>1. 0.3 0.3 1.0</diffuse>
+                    <specular>1. 0.3 0.3 1.0</specular>
+                    <emissive>1. 0.3 0.3 1.0</emissive>
+                </material>
             </visual>
         </gazebo>
         <link name="pince_g">
             <visual>
-            <!-- <origin xyz="-0.15 0 0" rpy="0 0 0"/> -->
-            <geometry>
-                <!-- <box size="0.7 0.05 0.2"/> -->
-                <box size="0.2 0.01 0.2"/>
-            </geometry>
-            <material name="Brown">
-                <color rgba="0.30 0.15 0.0 1.0"/>
-            </material>
-            </visual>
-            <collision>
-            <origin xyz="-0.15 0 0" rpy="0 0 0"/>
-            <geometry>
-                <!-- <box size="0.7 0.05 0.2"/> -->
-                <box size="0.2 0.01 0.2"/>
-            </geometry>
-            </collision>
-            <xacro:box_inertia m="0.00001" w="0.7" d="0.05" h="0.2"/>
+                <!-- <origin xyz="-0.15 0 0" rpy="0 0 0"/> -->
+                <geometry>
+                    <!-- <box size="0.7 0.05 0.2"/> -->
+                    <box size="0.2 0.01 0.2" />
+                </geometry>
+                <material name="Brown">
+                    <color rgba="0.30 0.15 0.0 1.0" />
+                </material>
+            </visual>
+            <collision>
+                <origin xyz="-0.15 0 0" rpy="0 0 0" />
+                <geometry>
+                    <!-- <box size="0.7 0.05 0.2"/> -->
+                    <box size="0.2 0.01 0.2" />
+                </geometry>
+            </collision>
+            <xacro:box_inertia m="0.00001" w="0.7" d="0.05" h="0.2" />
         </link>
         <joint name="pince_g_joint" type="fixed">
             <!-- <axis xyz="0 1 0"/> -->
             <!-- <origin xyz="0.25 -0.23 0" rpy="-1.5 0 ${-0.5 * pi}"/> -->
-            <origin xyz="-0.4 0.4 0" rpy="${0* pi} ${0* pi} ${(1/4) * pi}"/>
-            <parent link="segment_central"/>
-            <child link="pince_g"/>
-            <!-- <dynamics damping="0.0" friction="0.0"/> -->
-        </joint>
-<!--
-        <xacro:segment name="segment_g" x="0.3" y="0.01" z="0.2" joint_parent="segment_central" joint_origin_xyz="-0.25 0.46 0" joint_origin_rpy="0 ${0* pi} ${0 * pi}"/>
-        <xacro:segment name="fermeture_d" x="0.2" y="0.01" z="0.2" joint_parent="segment_central" joint_origin_xyz="-0.4 0.05 0" joint_origin_rpy="${0* pi} ${0* pi} ${(-1/4) * pi}"/> -->
-        <!-- <xacro:segment name="segment_d2" x="0.3" y="0.05" z="0.2" joint_parent="segment_d1" joint_origin_xyz="-0.30 -0.07 0" joint_origin_rpy="0 0 ${0.16 * pi}"/>
-        <xacro:segment name="segment_d3" x="0.3" y="0.05" z="0.2" joint_parent="segment_d2" joint_origin_xyz="-0.15 -0.1 0" joint_origin_rpy="0 0 ${-0.32* pi}"/>
-        <xacro:segment name="segment_g1" x="0.3" y="0.05" z="0.2" joint_parent="segment_central" joint_origin_xyz="0.25 -0.32 0" joint_origin_rpy="0 0 ${-0.16* pi}"/>
-        <xacro:segment name="segment_g2" x="0.3" y="0.05" z="0.2" joint_parent="segment_g1" joint_origin_xyz="0.30 -0.07 0" joint_origin_rpy="0 0 ${-0.16* pi}"/>
-        <xacro:segment name="segment_g3" x="0.3" y="0.05" z="0.2" joint_parent="segment_g2" joint_origin_xyz="0.15 -0.1 0" joint_origin_rpy="0 0 ${0.32* pi}"/>
-        <xacro:segment name="segment_triangled" x="0.3" y="0.05" z="0.2"  joint_parent="segment_central" joint_origin_xyz="-0.25 -0.12 0" joint_origin_rpy="0 0 ${-0.25* pi}"/>
-        <xacro:segment name="segment_triangleg" x="0.3" y="0.05" z="0.2"  joint_parent="segment_central" joint_origin_xyz="0.25 -0.12 0" joint_origin_rpy="0 0 ${0.25* pi}"/> -->
+            <origin xyz="-0.4 0.4 0" rpy="${0* pi} ${0* pi} ${(1/4) * pi}" />
+            <parent link="segment_central" />
+            <child link="pince_g" />
+            <!-- <dynamics damping="0.0" friction="0.0"/> -->
+        </joint>
+        <!--
+        <xacro:segment name="segment_g" x="0.3" y="0.01" z="0.2" joint_parent="segment_central"
+        joint_origin_xyz="-0.25 0.46 0" joint_origin_rpy="0 ${0* pi} ${0 * pi}"/>
+        <xacro:segment name="fermeture_d" x="0.2" y="0.01" z="0.2" joint_parent="segment_central"
+        joint_origin_xyz="-0.4 0.05 0" joint_origin_rpy="${0* pi} ${0* pi} ${(-1/4) * pi}"/> -->
+        <!-- <xacro:segment name="segment_d2" x="0.3" y="0.05" z="0.2" joint_parent="segment_d1"
+        joint_origin_xyz="-0.30 -0.07 0" joint_origin_rpy="0 0 ${0.16 * pi}"/>
+        <xacro:segment name="segment_d3" x="0.3" y="0.05" z="0.2" joint_parent="segment_d2"
+        joint_origin_xyz="-0.15 -0.1 0" joint_origin_rpy="0 0 ${-0.32* pi}"/>
+        <xacro:segment name="segment_g1" x="0.3" y="0.05" z="0.2" joint_parent="segment_central"
+        joint_origin_xyz="0.25 -0.32 0" joint_origin_rpy="0 0 ${-0.16* pi}"/>
+        <xacro:segment name="segment_g2" x="0.3" y="0.05" z="0.2" joint_parent="segment_g1"
+        joint_origin_xyz="0.30 -0.07 0" joint_origin_rpy="0 0 ${-0.16* pi}"/>
+        <xacro:segment name="segment_g3" x="0.3" y="0.05" z="0.2" joint_parent="segment_g2"
+        joint_origin_xyz="0.15 -0.1 0" joint_origin_rpy="0 0 ${0.32* pi}"/>
+        <xacro:segment name="segment_triangled" x="0.3" y="0.05" z="0.2"  joint_parent="segment_central"
+        joint_origin_xyz="-0.25 -0.12 0" joint_origin_rpy="0 0 ${-0.25* pi}"/>
+        <xacro:segment name="segment_triangleg" x="0.3" y="0.05" z="0.2"  joint_parent="segment_central"
+        joint_origin_xyz="0.25 -0.12 0" joint_origin_rpy="0 0 ${0.25* pi}"/> -->
     </xacro:macro>
 </robot>

Commit message: control ok

File: robot_description/src/description/robot_parts/collector2/collector.xacro (robot description, xacro)
@@ -138,5 +138,5 @@
             <!-- <axis xyz="0 1 0"/> -->
             <!-- <origin xyz="0.25 -0.23 0" rpy="-1.5 0 ${-0.5 * pi}"/> -->
-            <origin xyz="-0.4 0.05 0" rpy="${0* pi} ${0* pi} ${(-1/4) * pi}" />
+            <origin xyz="-0.4 0.05 0" rpy="${0* pi} ${0* pi} ${(-1/8) * pi}" />
             <parent link="segment_central" />
             <child link="pince_d" />
@@ -177,5 +177,5 @@
             <!-- <axis xyz="0 1 0"/> -->
             <!-- <origin xyz="0.25 -0.23 0" rpy="-1.5 0 ${-0.5 * pi}"/> -->
-            <origin xyz="-0.4 0.4 0" rpy="${0* pi} ${0* pi} ${(1/4) * pi}" />
+            <origin xyz="-0.4 0.4 0" rpy="${0* pi} ${0* pi} ${(1/8) * pi}" />
             <parent link="segment_central" />
             <child link="pince_g" />

Commit message: Done: La pince empeche sortie balle, premet d'attraper une balle et ne se réouvre pas toute seule

File: robot_description/src/description/robot_parts/collector2/collector.xacro (robot description, xacro)
@@ -19,8 +19,8 @@
         <link name="segment_central">
             <visual>
-                <origin xyz="-0.2 0 0" rpy="0 0 0" />
+                <origin xyz="-0.21 0 0" rpy="0 0 0" />
                 <geometry>
                     <!-- <box size="0.7 0.05 0.2"/> -->
-                    <box size="0.4 0.01 0.2" />
+                    <box size="0.42 0.01 0.2" />
                 </geometry>
                 <material name="Brown">
@@ -29,8 +29,8 @@
             </visual>
             <collision>
-                <origin xyz="-0.2 0 0" rpy="0 0 0" />
+                <origin xyz="-0.21 0 0" rpy="0 0 0" />
                 <geometry>
                     <!-- <box size="0.7 0.05 0.2"/> -->
-                    <box size="0.4 0.01 0.2" />
+                    <box size="0.42 0.01 0.2" />
                 </geometry>
             </collision>
@@ -81,5 +81,5 @@
                 <geometry>
                     <!-- <box size="0.7 0.05 0.2"/> -->
-                    <box size="0.3 0.01 0.2" />
+                    <box size="0.42 0.01 0.2" />
                 </geometry>
                 <material name="Brown">
@@ -88,8 +88,8 @@
             </visual>
             <collision>
-                <origin xyz="-0.15 0 0" rpy="0 0 0" />
+                <origin xyz="-0.21 0 0" rpy="0 0 0" />
                 <geometry>
                     <!-- <box size="0.7 0.05 0.2"/> -->
-                    <box size="0.3 0.01 0.2" />
+                    <box size="0.42 0.01 0.2" />
                 </geometry>
             </collision>
@@ -99,5 +99,5 @@
             <!-- <axis xyz="0 1 0"/> -->
             <!-- <origin xyz="0.25 -0.23 0" rpy="-1.5 0 ${-0.5 * pi}"/> -->
-            <origin xyz="-0.15 0.46 0" rpy="${0 * pi} ${(0) * pi} ${0 * pi}" />
+            <origin xyz="-0.21 0.46 0" rpy="${0 * pi} ${(0) * pi} ${0 * pi}" />
             <parent link="segment_central" />
             <child link="segment_g" />
@@ -120,5 +120,5 @@
                 <geometry>
                     <!-- <box size="0.7 0.05 0.2"/> -->
-                    <box size="0.175 0.01 0.2" />
+                    <box size="0.12 0.01 0.2" />
                 </geometry>
                 <material name="Brown">
@@ -130,5 +130,5 @@
                 <geometry>
                     <!-- <box size="0.7 0.05 0.2"/> -->
-                    <box size="0.175 0.01 0.2" />
+                    <box size="0.12 0.01 0.2" />
                 </geometry>
             </collision>
@@ -138,5 +138,5 @@
             <!-- <axis xyz="0 1 0"/> -->
             <!-- <origin xyz="0.25 -0.23 0" rpy="-1.5 0 ${-0.5 * pi}"/> -->
-            <origin xyz="-0.4 0.05 0" rpy="${0* pi} ${0* pi} ${(-1/5) * pi}" />
+            <origin xyz="-0.415 0.07 0" rpy="${0* pi} ${0* pi} ${(-1/2) * pi}" />
             <parent link="segment_central" />
             <child link="pince_d" />
@@ -159,5 +159,5 @@
                 <geometry>
                     <!-- <box size="0.7 0.05 0.2"/> -->
-                    <box size="0.175 0.01 0.2" />
+                    <box size="0.12 0.01 0.2" />
                 </geometry>
                 <material name="Brown">
@@ -169,5 +169,5 @@
                 <geometry>
                     <!-- <box size="0.7 0.05 0.2"/> -->
-                    <box size="0.175 0.01 0.2" />
+                    <box size="0.12 0.01 0.2" />
                 </geometry>
             </collision>
@@ -177,5 +177,5 @@
             <!-- <axis xyz="0 1 0"/> -->
             <!-- <origin xyz="0.25 -0.23 0" rpy="-1.5 0 ${-0.5 * pi}"/> -->
-            <origin xyz="-0.4 0.4 0" rpy="${0* pi} ${0* pi} ${(1/5) * pi}" />
+            <origin xyz="-0.415 0.39 0" rpy="${0* pi} ${0* pi} ${(1/2) * pi}" />
             <parent link="segment_central" />
             <child link="pince_g" />

Commit message: pince ouverte start + guidage corrige

File: robot_description/src/description/robot_parts/collector2/collector.xacro (robot description, xacro)
@@ -40,8 +40,8 @@
             <axis xyz="0 1 0" />
             <!-- <origin xyz="0.25 -0.23 0" rpy="-1.5 0 ${-0.5 * pi}"/> -->
-            <origin xyz="0.1 -0.23 0" rpy="${0 * pi} ${(-1/20) * pi} ${0 * pi}" />
+            <origin xyz="0.1 -0.23 0" rpy="${0 * pi} ${(-16/20) * pi} ${0 * pi}" />
             <parent link="base_link" />
             <child link="segment_central" />
-            <limit effort="1000000.0" lower="${(1/20) * pi}" upper="${(1+1/20) * pi}" velocity="30" />
+            <limit effort="1000000.0" lower="${(-4/20) * pi}" upper="${(-24/20) * pi}" velocity="30" />
             <dynamics damping="0.0" friction="10.0"/>
         </joint>
